File: FeuMontagne/FeuMontagne.kicad_pcb (KiCad board)
At the start: 2 copper layers, 73.4 x 41.9 mm, 26 parts, among them K1 CMD MAN, K10 F2, K11 R2, K12 R3, K13 R4, K2 A4, K3 A5, K4 A3, K5 12VAC, K6 RES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

Commit message: Corrections
Une erreur + changement des pastilles pour réalisation à la main plus facile + ajout du nom des cartes coté soudure
Other:
- board text added: "Feu Montagne"
